File: project-bed-light.kicad_pcb (KiCad board)
At the start: 2 copper layers, 58 x 56 mm, 24 parts, among them J1 2060-452_998-404, J2 WAGO_2060-453-998-404, J3 Conn_01x03_Pin, Q1 Q_Toshiba_SSM3J328R, U1 TPS62933, U2 Pink Panda v2.1.0

Commit message: pcb: add name
Other:
- board text added: "3.3V"
- board text added: "5V"
- board text added: "Julie Gervais 24 décembre 2025"

Commit message: pcb: couple little changes
Parts:
- R2: value Vchoice -> 52.3k
Routing:
- net GND: vias 35 -> 40
Changed lines of the file:
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@@
 			)
 		)
-		(property "Value" "Vchoice"
+		(property "Value" "52.3k"
 			(at 0 1.43 90)
 			(layer "F.Fab")
@@
 	)
 	(via
-		(at 67.25 60.5)
+		(at 67.25 60)
 		(size 0.6)
 		(drill 0.3)
@@
 	)
 	(via
-		(at 61.5 27)
+		(at 61 27)
 		(size 0.6)
 		(drill 0.3)
@@
 	)
 	(via
-		(at 76.5 27.75)
+		(at 77 27.75)
 		(size 0.6)
 		(drill 0.3)
@@
 	)
 	(via
-		(at 67.25 75.5)
+		(at 67.25 76)
 		(size 0.6)
 		(drill 0.3)
@@
 	)
 	(via
-		(at 68.700528 60.512186)
+		(at 68.75 60)
 		(size 0.6)
 		(drill 0.3)
@@
 	)
 	(via
-		(at 75.5 46)
+		(at 76 46)
 		(size 0.6)
 		(drill 0.3)
@@
 	)
 	(via
+		(at 70 45)
+		(size 0.6)
+		(drill 0.3)
+		(layers "F.Cu" "B.Cu")
+		(free yes)
+		(net 1)
+	)
+	(via
 		(at 22.5 38)
 		(size 0.6)
@@
 	)
 	(via
-		(at 45.25 29)
+		(at 45 29.14)
 		(size 0.6)
 		(drill 0.3)
@@
 	)
 	(via
-		(at 61.5 26.25)
+		(at 44.5 66.5)
 		(size 0.6)
 		(drill 0.3)
@@
 	)
 	(via
-		(at 68 60.5)
+		(at 61 26.25)
+		(size 0.6)
+		(drill 0.3)
+		(layers "F.Cu" "B.Cu")
+		(free yes)
+		(net 1)
+	)
+	(via
+		(at 68 60)
+		(size 0.6)
+		(drill 0.3)
+		(layers "F.Cu" "B.Cu")
+		(free yes)
+		(net 1)
+	)
+	(via
+		(at 43 66.5)
+		(size 0.6)
+		(drill 0.3)
+		(layers "F.Cu" "B.Cu")
+		(free yes)
+		(net 1)
+	)
+	(via
+		(at 70 46)
 		(size 0.6)
 		(drill 0.3)
@@
 	)
 	(via
-		(at 68 75.5)
+		(at 68 76)
 		(size 0.6)
 		(drill 0.3)
@@
 	)
 	(via
-		(at 75.5 44)
+		(at 76 44)
 		(size 0.6)
 		(drill 0.3)
@@
 	)
 	(via
-		(at 68.75 75.5)
+		(at 68.75 76)
 		(size 0.6)
 		(drill 0.3)
@@
 	)
 	(via
-		(at 76.5 27)
+		(at 77 27)
 		(size 0.6)
 		(drill 0.3)
@@
 	)
 	(via
-		(at 61.5 27.75)
+		(at 61 27.75)
 		(size 0.6)
 		(drill 0.3)
@@
 	)
 	(via
-		(at 75.5 45)
+		(at 76 45)
 		(size 0.6)
 		(drill 0.3)
@@
 	)
 	(via
-		(at 76.5 26.25)
+		(at 70 44)
+		(size 0.6)
+		(drill 0.3)
+		(layers "F.Cu" "B.Cu")
+		(free yes)
+		(net 1)
+	)
+	(via
+		(at 77 26.25)
 		(size 0.6)
 		(drill 0.3)
@@
 		(hatch edge 0.5)
 		(connect_pads
-			(clearance 0.2)
+			(clearance 0.5)
 		)
 		(min_thickness 0.2)
 		(filled_areas_thickness no)
 		(fill yes
-			(thermal_gap 0.2)
-			(thermal_bridge_width 0.2)
+			(thermal_gap 0.5)
+			(thermal_bridge_width 0.5)
 			(smoothing fillet)
 			(radius 0.5)
@@
 		(hatch edge 0.5)
 		(connect_pads
-			(clearance 0.2)
+			(clearance 0.5)
 		)
 		(min_thickness 0.2)
 		(filled_areas_thickness no)
 		(fill yes
-			(thermal_gap 0.2)
-			(thermal_bridge_width 0.2)
+			(thermal_gap 0.5)
+			(thermal_bridge_width 0.5)
 			(smoothing fillet)
 			(radius 0.5)
@@
 		(polygon
 			(pts
-				(xy 66 76) (xy 58 76) (xy 58 69) (xy 60 67) (xy 60 33) (xy 78 33) (xy 78 42) (xy 70 42) (xy 66 60)
+				(xy 66 76) (xy 58 76) (xy 58 69) (xy 60 69) (xy 60 33) (xy 78 33) (xy 78 42) (xy 69 42) (xy 66 60)
 			)
 		)
